File: logger.sch (KiCad schematic (older format))
At the start: 47 parts, among them IC1 ATMEGA1284P-A, P1 CONN_5X2, U1 LT1615-1, U2 AT45DB321D, U3 MCP6054, U4 MAX11612, U5 TPS7703X, U6 ADXL337, U7 LIS3DSH, X1 CRYSTAL

Commit message: General layout/grounding tweaks, DC-DC layout improved, ADC set up for Vdd as ref, switchable 3v3_Analog for lower standby power, reset circuitry redone, Footprint fixes, better silkscreen.
Parts:
- removed U2: AT45DB321D, SO8E, symbol AT45DB321D
- added C26: C, SM0603_Capa, symbol C
- added C27, C28: 1u, SM0603_Capa, symbol CSMALL
- added C29: 10u, SM0805, symbol C
- added C30: 1u, symbol C
- added L5: 10u, SM2010, symbol INDUCTOR_SMALL
- added Q1: MOS_P, symbol MOS_P
- added R20: 1M, symbol R
- added R30: 1, SM0603, symbol R
- added R31: 1k, symbol R
- added U2: SST25VF064C, symbol SST25VF064C
- C11, C12, C13, C14, C5, C9: footprint SM0603_Capa -> SM0805
- C23, C24, C25: footprint ~ -> SM0603_Capa
- D1: footprint SM0603 -> SOD323
- U4: value MAX11612 -> MAX11613
Connections:
- net labels added: 3V3_Analog, 3V3_Analog_Unswitched, Vmon
- wire segments 247 -> 274
Other:
- moved on the sheet: C14
